Commit message: extend more

File: sr_description/hand/xacro/thumb/thdistal.urdf.xacro (robot description, xacro)
@@ -192,5 +192,5 @@
         <origin xyz="0 0 0.032" rpy="0 0 ${-M_PI/2}" />
         <axis xyz="1 0 0" />
-        <limit lower="-0.2618" upper="${90.0*M_PI/180}" effort="1.0"
+        <limit lower="-0.349" upper="${90.0*M_PI/180}" effort="1.0"
         velocity="4.0" />
         <dynamics damping="0.2" />

File: sr_description/hand/xacro/thumb/thproximal.urdf.xacro (robot description, xacro)
@@ -43,5 +43,5 @@
       <origin xyz="0 0 0" rpy="0 0 0" />
       <axis xyz="${reflect} 0 0" />
-      <limit lower="0.0" upper="${70/180*M_PI}" effort="3"
+      <limit lower="0.0" upper="${78/180*M_PI}" effort="3"
       velocity="4.0" />
       <dynamics damping="0.2" />
