Commit message: adding param part 1

File: sr_description/hand/xacro/ff_biotac_hand.urdf.xacro (robot description, xacro)
@@ -18,5 +18,5 @@
   <!-- prefix can be anything but usually is "r_" or  "l_" for right and left hands distinction -->
   <xacro:macro name="shadowhand"
-  params="muscletrans muscle bio bt_sp ubi eli reflect prefix">
+  params="muscletrans muscle bio bt_sp ubi eli reflect prefix extended_limits">
     <!-- Forearm -->
     <xacro:forearm muscle="${muscle}" prefix="${prefix}" />

File: sr_description/hand/xacro/finger/fingers.urdf.xacro (robot description, xacro)
@@ -17,6 +17,7 @@
   <!-- joint_prefix prepends fingername to the joint names -->
   <!-- parent is the parent link for the first joint -->
+  <!-- extended_limits is true if using the extended range of this joint -->
   <xacro:macro name="finger"
-  params="muscletrans lf bio bt_sp ubi eli reflect prefix link_prefix joint_prefix parent *origin *axis">
+  params="muscletrans lf bio bt_sp ubi eli reflect prefix link_prefix joint_prefix parent *origin *axis extended_limits:='false'">
     <!-- Little finger special case -->
     <xacro:if value="${lf}">

File: sr_description/hand/xacro/finger/proximal/proximal.urdf.xacro (robot description, xacro)
@@ -13,6 +13,7 @@
   <!-- joint_prefix prepends fingername to the joint names -->
   <!-- parent is the parent link for the joint -->
+  <!-- extended_limits is true if using the extended range of this joint -->
   <xacro:macro name="proximal"
-  params="muscle prefix link_prefix joint_prefix parent">
+  params="muscle prefix link_prefix joint_prefix parent extended_limits">
     <link name="${prefix}${link_prefix}proximal">
       <inertial>
@@ -42,6 +43,12 @@
       <origin xyz="0 0 0" rpy="0 0 0" />
       <axis xyz="1 0 0" />
-      <limit lower="-${15.0*M_PI/180}" upper="${M_PI/2}" effort="2"
-      velocity="2.0" />
+      <xacro:if value="${extended_limits}">
+		<limit lower="-${15.0*M_PI/180}" upper="${M_PI/2}" effort="2"
+        velocity="2.0" />
+      </xacro:if>
+      <xacro:unless value="${extended_limits}">
+        <limit lower="0" upper="${M_PI/2}" effort="2"
+        velocity="2.0" />
+      </xacro:unless>
       <dynamics damping="0.1" />
     </joint>

File: sr_description/hand/xacro/full_hand.urdf.xacro (robot description, xacro)
@@ -19,5 +19,5 @@
   <!-- lf is true if we want a little finger, false otherwise -->
   <xacro:macro name="shadowhand"
-  params="muscletrans muscle hand_type:='hand_e' bio bt_sp ubi eli reflect prefix lf cable_mesh:='false'">
+  params="muscletrans muscle hand_type:='hand_e' bio bt_sp ubi eli reflect prefix lf extended_limits cable_mesh:='false'">
     <!--xacro:property name="hand_type" value="hand_e"/-->
     <!-- Forearm -->

File: sr_description/hand/xacro/hand_E_no_mf_rf.urdf.xacro (robot description, xacro)
@@ -19,5 +19,5 @@
   <!-- lf is true if we want a little finger, false otherwise -->
   <xacro:macro name="shadowhand"
-  params="muscletrans muscle bio bt_sp ubi eli reflect prefix lf">
+  params="muscletrans muscle bio bt_sp ubi eli reflect prefix lf extended_limits">
     <!-- Forearm -->
     <xacro:forearm muscle="${muscle}" prefix="${prefix}" />

File: sr_description/hand/xacro/hand_lite.urdf.xacro (robot description, xacro)
@@ -18,5 +18,5 @@
   <!-- prefix can be anything but usually is "r_" or  "l_" for right and left hands distinction -->
   <xacro:macro name="shadowhand"
-  params="muscletrans muscle bio bt_sp ubi eli reflect prefix extra_lite  cable_mesh:='false'">
+  params="muscletrans muscle bio bt_sp ubi eli reflect prefix extended_limits extra_lite cable_mesh:='false'">
     <!-- Forearm -->
     <xacro:forearm muscle="${muscle}" prefix="${prefix}" cable_mesh="${cable_mesh}"/>

File: sr_description/hand/xacro/one_finger_unit.urdf.xacro (robot description, xacro)
@@ -15,5 +15,5 @@
   <!-- prefix can be anything but usually is "r_" or  "l_" for right and left hands distinction -->
   <xacro:macro name="shadowhand"
-  params="muscletrans muscle bio bt_sp ubi eli reflect prefix">
+  params="muscletrans muscle bio bt_sp ubi eli reflect prefix extended_limits">
     <!-- Forearm -->
     <xacro:forearm muscle="${muscle}" prefix="${prefix}" />

File: sr_description/hand/xacro/th_ff_rf_ellipsoid_hand.urdf.xacro (robot description, xacro)
@@ -18,5 +18,5 @@
   <!-- prefix can be anything but usually is "r_" or  "l_" for right and left hands distinction -->
   <xacro:macro name="shadowhand"
-  params="muscletrans muscle bio bt_sp ubi eli reflect prefix">
+  params="muscletrans muscle bio bt_sp ubi eli reflect prefix extended_limits">
     <!-- Forearm -->
     <xacro:forearm muscle="${muscle}" prefix="${prefix}" />

File: sr_description/hand/xacro/three_biotac_fingers_hand.urdf.xacro (robot description, xacro)
@@ -18,5 +18,5 @@
   <!-- prefix can be anything but usually is "r_" or  "l_" for right and left hands distinction -->
   <xacro:macro name="shadowhand"
-  params="muscletrans muscle bio bt_sp ubi eli reflect prefix">
+  params="muscletrans muscle bio bt_sp ubi eli reflect prefix extended_limits">
     <!-- Forearm -->
     <xacro:forearm muscle="${muscle}" prefix="${prefix}" />

File: sr_description/hand/xacro/three_fingers_hand.urdf.xacro (robot description, xacro)
@@ -18,5 +18,5 @@
   <!-- prefix can be anything but usually is "r_" or  "l_" for right and left hands distinction -->
   <xacro:macro name="shadowhand"
-  params="muscletrans muscle bio bt_sp ubi eli reflect prefix">
+  params="muscletrans muscle bio bt_sp ubi eli reflect prefix extended_limits">
     <!-- Forearm -->
     <xacro:forearm muscle="${muscle}" prefix="${prefix}" />

File: sr_description/hand/xacro/three_fingers_hand_RF.urdf.xacro (robot description, xacro)
@@ -18,5 +18,5 @@
   <!-- prefix can be anything but usually is "r_" or  "l_" for right and left hands distinction -->
   <xacro:macro name="shadowhand"
-  params="muscletrans muscle bio bt_sp ubi eli reflect prefix">
+  params="muscletrans muscle bio bt_sp ubi eli reflect prefix extended_limits">
     <!-- Forearm -->
     <xacro:forearm muscle="${muscle}" prefix="${prefix}" />

File: sr_description/hand/xacro/thumb/thdistal.urdf.xacro (robot description, xacro)
@@ -15,6 +15,7 @@
   <!-- prefix can be anything but usually is "r_" or  "l_" for right and left hands distinction -->
   <!-- parent is the parent link for the first joint -->
+  <!-- extended_limits is true if using the extended range of this joint -->
   <xacro:macro name="thdistal"
-  params="muscle bio bt_sp ubi eli prefix parent">
+  params="muscle bio bt_sp ubi eli prefix parent extended_limits">
     <xacro:if value="${bio}">
       <!--    BIOTAC -->

File: sr_description/robots/arm_and_hand_motor.urdf.xacro (robot description, xacro)
@@ -17,4 +17,4 @@
   </joint>
   <xacro:shadowhand muscletrans="false" muscle="false" bio="false" bt_sp="false"
-  ubi="false" eli="false" reflect="1.0" prefix="rh_" lf="true" />
+  ubi="false" eli="false" reflect="1.0" prefix="rh_" lf="true" extended_limits:="false" />
 </robot>

File: sr_description/robots/arm_and_hand_motor_biotac.urdf.xacro (robot description, xacro)
@@ -17,4 +17,4 @@
   </joint>
   <xacro:shadowhand muscletrans="false" muscle="false" bio="true" bt_sp="false"
-  ubi="false" eli="false" reflect="1.0" prefix="rh_" lf="true" />
+  ubi="false" eli="false" reflect="1.0" prefix="rh_" lf="true" extended_limits:="false" />
 </robot>

File: sr_description/robots/arm_and_hand_motor_ellipsoid.urdf.xacro (robot description, xacro)
@@ -17,4 +17,4 @@
   </joint>
   <xacro:shadowhand muscletrans="false" muscle="false" bio="false" bt_sp="false"
-  ubi="false" eli="true" reflect="1.0" prefix="rh_" lf="true" />
+  ubi="false" eli="true" reflect="1.0" prefix="rh_" lf="true" extended_limits:="false" />
 </robot>

File: sr_description/robots/arm_and_hand_motor_three_finger.urdf.xacro (robot description, xacro)
@@ -17,4 +17,4 @@
   </joint>
   <xacro:shadowhand muscletrans="false" muscle="false" bio="false" bt_sp="false"
-  ubi="false" eli="false" reflect="1.0" prefix="rh_" />
+  ubi="false" eli="false" reflect="1.0" prefix="rh_" extended_limits:="false" />
 </robot>

File: sr_description/robots/arm_and_hand_muscle.urdf.xacro (robot description, xacro)
@@ -17,4 +17,4 @@
   </joint>
   <xacro:shadowhand muscletrans="false" muscle="true" bio="false" bt_sp="false"
-  ubi="false" eli="false" reflect="1.0" prefix="rh_" lf="true" />
+  ubi="false" eli="false" reflect="1.0" prefix="rh_" lf="true" extended_limits:="false" />
 </robot>

File: sr_description/robots/arm_and_hand_muscle_biotac.urdf.xacro (robot description, xacro)
@@ -17,4 +17,4 @@
   </joint>
   <xacro:shadowhand muscletrans="false" muscle="true" bio="true" bt_sp="false"
-  ubi="false" eli="false" reflect="1.0" prefix="rh_" lf="true" />
+  ubi="false" eli="false" reflect="1.0" prefix="rh_" lf="true" extended_limits:="false" />
 </robot>

File: sr_description/robots/arm_and_sr_one_finger_motor.urdf.xacro (robot description, xacro)
@@ -20,4 +20,4 @@
   </joint>
   <xacro:shadowhand muscletrans="false" muscle="false" bio="false" bt_sp="false"
-  ubi="false" eli="false" reflect="1.0" prefix="rh_" />
+  ubi="false" eli="false" reflect="1.0" prefix="rh_" extended_limits:="false" />
 </robot>

File: sr_description/robots/bimanual_shadowhand_extra_lite.urdf.xacro (robot description, xacro)
@@ -19,4 +19,4 @@
   </joint>
   <xacro:shadowhand muscletrans="false" muscle="false" bio="false" bt_sp="false"
-                    ubi="false" eli="false" reflect="-1.0" prefix="lh_" extra_lite="true" />
+                    ubi="false" eli="false" reflect="-1.0" prefix="lh_" extended_limits:="false" extra_lite="true" />
 </robot>
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